Commit message: tweak platform base visuals

File: arondite/assets/platform.urdf (robot description, URDF)
Before this commit: robot platform, 4 links, 3 joints
Links:
- link base_link: geometry visual box size=0.1 0.1 0.1

Commit message: Use multiple links to create textures

File: arondite/assets/platform.urdf (robot description, URDF)
Before this commit: robot platform, 4 links, 3 joints
Links:
- added link horizontal; visual box size=2.5 0.2 0.01
- added link vertical; visual box size=0.2 2.5 0.01
- link helipad_yrot_link: geometry collision box size=2.5 2.5 0.01; visual box size=2.5 2.5 0.01
Joints:
- added joint helipad_to_horizontal: type fixed, parent helipad_yrot_link, child horizontal, origin xyz=0.0 0.0 0.0001
- added joint helipad_to_vertical: type fixed, parent helipad_yrot_link, child vertical, origin xyz=0.0 0.0 0.0001
